Commit message: robot configuration

File: src/my_robot_pkg/description/robot.urdf.xacro (robot description, xacro)
@@ -1,6 +1,4 @@
-<?<?xml version="1.0"?>
-<<robot xmlns:xacro="https://www.ros.org/wiki/xacro" name="robot">
-    <!-- Example link -->
-    <<link name="base_link">
-    </link>
+<?xml version="1.0"?>
+<robot xmlns:xacro="https://www.ros.org/wiki/xacro" name="robot">
+    <xacro:include filename="robot_core.xacro"/>
 </robot>
