Commit message: create urdf

File: install/my_robot_pkg/share/my_robot_pkg/description/robot_core.xacro (robot description, xacro)
@@ -1,5 +1,5 @@
 <?xml version="1.0"?>
 <robot xmlns:xacro="https://www.ros.org/wiki/xacro" name="robot">
-    <xacro:includ filename="inertial_macros.xacro"/>
+    <xacro:include filename="inertial_macros.xacro"/>
     <material name = "white">
         <color rgba="1 1 1 1"/>
@@ -37,5 +37,5 @@
             </geometry>
         </collision>
-        <xacro:inertial_box mass="0.5" x="0.3" y="0.3" z="0.15"/>
+        <xacro:inertial_box mass="0.5" x="0.3" y="0.3" z="0.15">
             <origin xyz="0.15 0 0.075" rpy="0 0 0"/>
         </xacro:inertial_box>
@@ -61,5 +61,5 @@
         </collision>
         <xacro:inertial_cylinder mass="0.1" length="0.04" radius="0.05">
-            <origin xyz="0.0 0.0 0.0" rpy="0.0 0.0 0.0"/>
+            <origin xyz="0 0 0" rpy="0 0 0"/>
         </xacro:inertial_cylinder>
     </link>
@@ -84,5 +84,5 @@
         </collision>
         <xacro:inertial_cylinder mass="0.1" length="0.04" radius="0.05">
-            <origin xyz="0.0 0.0 0.0" rpy="0.0 0.0 0.0"/>
+            <origin xyz="0 0 0" rpy="0 0 0"/>
         </xacro:inertial_cylinder>
     </link>

File: src/my_robot_pkg/description/inertial_macros.xacro (robot description, xacro)
@@ -1,3 +1,32 @@
 <?xml version="1.0"?>
 <robot xmlns:xacro="https://www.ros.org/wiki/xacro">
+    <!-- Specify some standard inertial calculations https://en.wikipedia.org/wiki/List_of_moments_of_inertia -->
+    <!-- These make use of xacro's mathematical functionality -->
+    <xacro:macro name="inertial_sphere" params="mass radius *origin">
+        <inertial>
+            <xacro:insert_block name="origin"/>
+            <mass value="${mass}"/>
+            <inertia ixx = "${(2/5) * mass * (radius * radius)}" ixy = "0.0" ixz = "0.0"
+                    iyy = "${(2/5) * mass * (radius * radius)}" iyz = "0.0"
+                    izz = "${(2/5) * mass * (radius * radius)}"/>
+        </inertial>
+    </xacro:macro>
+    <xacro:macro name = "inertial_box" params = "mass x y z *origin">
+        <inertial>
+            <xacro:insert_block name = "origin"/>
+            <mass value="${mass}"/>
+            <inertia ixx = "${(1/12) * mass * (y*y + z*z)}" ixy = "0.0" ixz = "0.0"
+                    iyy = "${(1/12) * mass * (x*x + z*z)}" iyz = "0.0"
+                    izz = "${(1/12) * mass * (x*x + y*y)}"/>
+        </inertial>
+    </xacro:macro>
+    <xacro:macro name = "inertial_cylinder" params = "mass length radius *origin">
+        <inertial>
+            <xacro:insert_block name = "origin"/>
+            <mass value = "${mass}"/>
+            <inertia ixx = "${(1/12) * mass * (3*radius*radius + length*length)}" ixy = "0.0" ixz = "0.0"
+                    iyy = "${(1/12) * mass * (3*radius*radius + length*length)}" iyz = "0.0"
+                    izz = "${(1/12) * mass * (radius*radius)}"/>
+        </inertial>
+    </xacro:macro>
 </robot>

Commit message: gazebo launch

File: install/my_robot_pkg/share/my_robot_pkg/description/robot_core.xacro (robot description, xacro)
@@ -14,5 +14,5 @@
         <color rgba="0 0 0 1"/>
     </material>
-    <!-- CHASE LINK -->
+    <!-- BASE LINK -->
     <link name="base_link">
     </link>
@@ -41,4 +41,7 @@
         </xacro:inertial_box>
     </link>
+    <gazebo reference = "chassis">
+        <material name="Gazebo/White"/>
+    </gazebo>
     <!-- LEFT WHEEL LINK -->
     <joint name="left_wheel_joint" type="continuous">
@@ -64,4 +67,7 @@
         </xacro:inertial_cylinder>
     </link>
+    <gazebo reference = "left_wheel">
+        <material name="Gazebo/Blue"/>
+    </gazebo>
     <!-- RIGHT WHEEL -->
     <joint name="right_wheel_joint" type="continuous">
@@ -87,4 +93,7 @@
         </xacro:inertial_cylinder>
     </link>
+    <gazebo reference="right_wheel">
+        <material name="Gazebo/Blue"/>
+    </gazebo>
     <!-- CASTER WHEEL LINK -->
     <joint name="caster_wheel_joint" type="fixed">
@@ -109,3 +118,6 @@
         </xacro:inertial_sphere>
     </link>
+    <gazebo reference="caster_wheel">
+        <material name="Gazebo/Black"/>
+    </gazebo>
 </robot>

File: src/my_robot_pkg/description/robot_core.xacro (robot description, xacro)
@@ -14,5 +14,5 @@
         <color rgba="0 0 0 1"/>
     </material>
-    <!-- CHASE LINK -->
+    <!-- BASE LINK -->
     <link name="base_link">
     </link>
@@ -41,4 +41,9 @@
         </xacro:inertial_box>
     </link>
+    <gazebo reference = "chassis">
+        <material>
+            Gazebo/White
+        </material>
+    </gazebo>
     <!-- LEFT WHEEL LINK -->
     <joint name="left_wheel_joint" type="continuous">
@@ -64,4 +69,9 @@
         </xacro:inertial_cylinder>
     </link>
+    <gazebo reference = "left_wheel">
+        <material>
+            Gazebo/Blue
+        </material>
+    </gazebo>
     <!-- RIGHT WHEEL -->
     <joint name="right_wheel_joint" type="continuous">
@@ -87,4 +97,9 @@
         </xacro:inertial_cylinder>
     </link>
+    <gazebo reference="right_wheel">
+        <material>
+            Gazebo/Blue
+        </material>
+    </gazebo>
     <!-- CASTER WHEEL LINK -->
     <joint name="caster_wheel_joint" type="fixed">
@@ -109,3 +124,8 @@
         </xacro:inertial_sphere>
     </link>
+    <gazebo reference="caster_wheel">
+        <material>
+            Gazebo/Black
+        </material>
+    </gazebo>
 </robot>
