Commit message: gazebo new

File: install/my_robot_pkg/share/my_robot_pkg/description/robot.urdf.xacro (robot description, xacro)
@@ -2,3 +2,4 @@
 <robot xmlns:xacro="https://www.ros.org/wiki/xacro" name="robot">
     <xacro:include filename="robot_core.xacro"/>
+    <xacro:include filename="gazebo_control.xacro"/>
 </robot>

File: install/my_robot_pkg/share/my_robot_pkg/description/robot_core.xacro (robot description, xacro)
@@ -42,5 +42,7 @@
     </link>
     <gazebo reference = "chassis">
-        <material name="Gazebo/White"/>
+        <material>
+            Gazebo/White
+        </material>
     </gazebo>
     <!-- LEFT WHEEL LINK -->
@@ -68,5 +70,7 @@
     </link>
     <gazebo reference = "left_wheel">
-        <material name="Gazebo/Blue"/>
+        <material>
+            Gazebo/Blue
+        </material>
     </gazebo>
     <!-- RIGHT WHEEL -->
@@ -94,5 +98,7 @@
     </link>
     <gazebo reference="right_wheel">
-        <material name="Gazebo/Blue"/>
+        <material>
+            Gazebo/Blue
+        </material>
     </gazebo>
     <!-- CASTER WHEEL LINK -->
@@ -119,5 +125,7 @@
     </link>
     <gazebo reference="caster_wheel">
-        <material name="Gazebo/Black"/>
+        <material>
+            Gazebo/Black
+        </material>
     </gazebo>
 </robot>

File: src/my_robot_pkg/description/robot.urdf.xacro (robot description, xacro)
@@ -2,3 +2,4 @@
 <robot xmlns:xacro="https://www.ros.org/wiki/xacro" name="robot">
     <xacro:include filename="robot_core.xacro"/>
+    <xacro:include filename="gazebo_control.xacro"/>
 </robot>

File: src/my_robot_pkg/description/robot_core.xacro (robot description, xacro)
@@ -128,4 +128,6 @@
             Gazebo/Black
         </material>
+        <mu1 value="0.001"/>
+        <mu2 value="0.001"/>
     </gazebo>
 </robot>
