Commit message: drone

File: install/my_robot_pkg/share/my_robot_pkg/description/drone.urdf.xacro (robot description, xacro)
@@ -2,4 +2,5 @@
 <robot xmlns:xacro="http://www.ros.org/wiki/xacro" name="drone">\
     <xacro:include filename = "inertial_macros.xacro"/>
+    <xacro:include filename = "drone_macros.xacro"/>
     <!-- MATERIAL -->
     <material name = "white">
@@ -20,6 +21,7 @@
     <xacro:property name = "base_height" value = "0.1"/>
     <xacro:property name = "rotor_radius" value = "0.05"/>
-    <xacro:property name = "rotor_length" value = "0.04"/>
+    <xacro:property name = "rotor_length" value = "0.05"/>
     <xacro:property name = "mass" value = "1.0"/>
+    <xacro:property name = "wing_pos" value = "${base_height/2+0.02}"/>
     <!-- BASE_LINK -->
     <link name="base_link">
@@ -52,123 +54,19 @@
         Gazebo/White
     </gazebo>
-    <!-- Wing 1 -->
-    <joint name="wing1_joint" type="fixed">
-        <parent link="body_link"/>
-        <child link="wing1"/>
-        <origin xyz="0 0 0" rpy="0 0 ${pi/4}"/>
-    </joint>
-    <link name="wing1">
-        <visual>
-            <origin xyz="0.3 0.0 ${base_height/2}"/>
-            <geometry>
-                <box size="0.3 0.08 0.03"/>
-            </geometry>
-            <material name="orange"/>
-        </visual>
-        <collision>
-            <origin xyz="0.3 0.0 ${base_height/2}"/>
-            <geometry>
-                <box size="0.3 0.08 0.03"/>
-            </geometry>
-        </collision>
-    </link>
+    <!-- Bar 1 -->
+    <xacro:bar name="bar1" parent="body_link" angle="${pi/4}" pos="0.3 0 ${wing_pos}" size="0.3 0.08 0.03"></xacro:bar>
     <!-- Rotor 1 -->
-    <joint name="rotor1_joint" type="continuous">
-        <parent link="wing1"/>
-        <child link="rotor1"/>
-        <origin xyz="${0.45-rotor_radius} 0.0 ${base_height/2 +0.015}"/>
-        <axis xyz="0 0 1"/>
-    </joint>
-    <link name="rotor1">
-    </link>
-    <!-- Wing 2 -->
-    <joint name="wing2_joint" type="fixed">
-        <parent link="body_link"/>
-        <child link="wing2"/>
-        <origin xyz="0 0 0" rpy="0 0 ${3*pi/4}"/>
-    </joint>
-    <link name="wing2">
-        <visual>
-            <origin xyz="0.3 0.0 ${base_height/2}"/>
-            <geometry>
-                <box size="0.3 0.08 0.03"/>
-            </geometry>
-            <material name="orange"/>
-        </visual>
-        <collision>
-            <origin xyz="0.3 0.0 ${base_height/2}"/>
-            <geometry>
-                <box size="0.3 0.08 0.03"/>
-            </geometry>
-        </collision>
-    </link>
+    <xacro:rotor num="1" parent="bar1" radius="${rotor_radius}" length="${rotor_length}" wing_pos="${wing_pos}"></xacro:rotor>
+    <!-- Bar 2 -->
+    <xacro:bar name="bar2" parent="body_link" angle="${3*pi/4}" pos="0.3 0 ${wing_pos}" size="0.3 0.08 0.03"></xacro:bar>
     <!-- Rotor 2 -->
-    <joint name="rotor2_joint" type="continuous">
-        <parent link="wing2"/>
-        <child link="rotor2"/>
-        <origin xyz="${0.45-rotor_radius} 0.0 ${base_height/2 +0.015}"/>
-        <axis xyz="0 0 -1"/>
-    </joint>
-    <link name="rotor2">
-    </link>
-    <!-- Wing 3 -->
-    <joint name="wing3_joint" type="fixed">
-        <parent link="body_link"/>
-        <child link="wing3"/>
-        <origin xyz="0 0 0" rpy="0 0 ${-3*pi/4}"/>
-    </joint>
-    <link name="wing3">
-        <visual>
-            <origin xyz="0.3 0.0 ${base_height/2}"/>
-            <geometry>
-                <box size="0.3 0.08 0.03"/>
-            </geometry>
-            <material name="orange"/>
-        </visual>
-        <collision>
-            <origin xyz="0.3 0.0 ${base_height/2}"/>
-            <geometry>
-                <box size="0.3 0.08 0.03"/>
-            </geometry>
-        </collision>
-    </link>
+    <xacro:rotor num="2" parent="bar2" radius="${rotor_radius}" length="${rotor_length}" wing_pos="${wing_pos}"></xacro:rotor>
+    <!-- Bar 3 -->
+    <xacro:bar name="bar3" parent="body_link" angle="${-3*pi/4}" pos="0.3 0 ${wing_pos}" size="0.3 0.08 0.03"></xacro:bar>
     <!-- Rotor 3 -->
-    <joint name="rotor3_joint" type="continuous">
-        <parent link="wing3"/>
-        <child link="rotor3"/>
-        <origin xyz="${0.45-rotor_radius} 0.0 ${base_height/2 +0.015}"/>
-        <axis xyz="0 0 1"/>
-    </joint>
-    <link name="rotor3">
-    </link>
-    <!-- Wing 4 -->
-    <joint name="wing4_joint" type="fixed">
-        <parent link="body_link"/>
-        <child link="wing4"/>
-        <origin xyz="0 0 0" rpy="0 0 ${-pi/4}"/>
-    </joint>
-    <link name="wing4">
-        <visual>
-            <origin xyz="0.3 0.0 ${base_height/2}"/>
-            <geometry>
-                <box size="0.3 0.08 0.03"/>
-            </geometry>
-            <material name="orange"/>
-        </visual>
-        <collision>
-            <origin xyz="0.3 0.0 ${base_height/2}"/>
-            <geometry>
-                <box size="0.3 0.08 0.03"/>
-            </geometry>
-        </collision>
-    </link>
+    <xacro:rotor num="3" parent="bar3" radius="${rotor_radius}" length="${rotor_length}" wing_pos="${wing_pos}"></xacro:rotor>
+    <!-- Bar 4 -->
+    <xacro:bar name="bar4" parent="body_link" angle="${-pi/4}" pos="0.3 0 ${wing_pos}" size="0.3 0.08 0.03"></xacro:bar>
     <!-- Rotor 4 -->
-    <joint name="rotor4_joint" type="continuous">
-        <parent link="wing4"/>
-        <child link="rotor4"/>
-        <origin xyz="${0.45-rotor_radius} 0.0 ${base_height/2 +0.015}"/>
-        <axis xyz="0 0 -1"/>
-    </joint>
-    <link name="rotor4">
-    </link>
+    <xacro:rotor num="4" parent="bar4" radius="${rotor_radius}" length="${rotor_length}" wing_pos="${wing_pos}"></xacro:rotor>
 </robot>

Commit message: fix drone.urdf

File: install/my_robot_pkg/share/my_robot_pkg/description/drone.urdf.xacro (robot description, xacro)
@@ -1,4 +1,4 @@
 <?xml version="1.0"?>
-<robot xmlns:xacro="http://www.ros.org/wiki/xacro" name="drone">\
+<robot xmlns:xacro="http://www.ros.org/wiki/xacro" name="drone">
     <xacro:include filename = "inertial_macros.xacro"/>
     <xacro:include filename = "drone_macros.xacro"/>
@@ -55,18 +55,18 @@
     </gazebo>
     <!-- Bar 1 -->
-    <xacro:bar name="bar1" parent="body_link" angle="${pi/4}" pos="0.3 0 ${wing_pos}" size="0.3 0.08 0.03"></xacro:bar>
+    <xacro:bar name="bar1" parent="body_link" angle="${pi/4}" pos="0.3 0 ${wing_pos}" size="0.3 0.08 0.03" mass="${mass}"></xacro:bar>
     <!-- Rotor 1 -->
-    <xacro:rotor num="1" parent="bar1" radius="${rotor_radius}" length="${rotor_length}" wing_pos="${wing_pos}"></xacro:rotor>
+    <xacro:rotor num="1" parent="bar1" radius="${rotor_radius}" length="${rotor_length}" wing_pos="${wing_pos}" mass="${mass}"></xacro:rotor>
     <!-- Bar 2 -->
-    <xacro:bar name="bar2" parent="body_link" angle="${3*pi/4}" pos="0.3 0 ${wing_pos}" size="0.3 0.08 0.03"></xacro:bar>
+    <xacro:bar name="bar2" parent="body_link" angle="${3*pi/4}" pos="0.3 0 ${wing_pos}" size="0.3 0.08 0.03" mass="${mass}"></xacro:bar>
     <!-- Rotor 2 -->
-    <xacro:rotor num="2" parent="bar2" radius="${rotor_radius}" length="${rotor_length}" wing_pos="${wing_pos}"></xacro:rotor>
+    <xacro:rotor num="2" parent="bar2" radius="${rotor_radius}" length="${rotor_length}" wing_pos="${wing_pos}" mass="${mass}"></xacro:rotor>
     <!-- Bar 3 -->
-    <xacro:bar name="bar3" parent="body_link" angle="${-3*pi/4}" pos="0.3 0 ${wing_pos}" size="0.3 0.08 0.03"></xacro:bar>
+    <xacro:bar name="bar3" parent="body_link" angle="${-3*pi/4}" pos="0.3 0 ${wing_pos}" size="0.3 0.08 0.03" mass="${mass}"></xacro:bar>
     <!-- Rotor 3 -->
-    <xacro:rotor num="3" parent="bar3" radius="${rotor_radius}" length="${rotor_length}" wing_pos="${wing_pos}"></xacro:rotor>
+    <xacro:rotor num="3" parent="bar3" radius="${rotor_radius}" length="${rotor_length}" wing_pos="${wing_pos}" mass="${mass}"></xacro:rotor>
     <!-- Bar 4 -->
-    <xacro:bar name="bar4" parent="body_link" angle="${-pi/4}" pos="0.3 0 ${wing_pos}" size="0.3 0.08 0.03"></xacro:bar>
+    <xacro:bar name="bar4" parent="body_link" angle="${-pi/4}" pos="0.3 0 ${wing_pos}" size="0.3 0.08 0.03" mass="${mass}"></xacro:bar>
     <!-- Rotor 4 -->
-    <xacro:rotor num="4" parent="bar4" radius="${rotor_radius}" length="${rotor_length}" wing_pos="${wing_pos}"></xacro:rotor>
+    <xacro:rotor num="4" parent="bar4" radius="${rotor_radius}" length="${rotor_length}" wing_pos="${wing_pos}" mass="${mass}"></xacro:rotor>
 </robot>

File: install/my_robot_pkg/share/my_robot_pkg/description/drone_macros.xacro (robot description, xacro)
@@ -1,6 +1,8 @@
 <?xml version="1.0"?>
 <robot xmlns:xacro="http://www.ros.org/wiki/xacro">
+    <xacro:include filename="inertial_macros.xacro"/>
+    <xacro:property name = "mass" value = "1.0"/>
     <!-- Bar -->
-    <xacro:macro name="bar" params="name parent angle pos size ">
+    <xacro:macro name="bar" params="name parent angle pos size mass">
         <joint name="${name}_joint" type="fixed">
             <parent link="${parent}"/>
@@ -22,8 +24,16 @@
                 </geometry>
             </collision>
+            <xacro:inertial_box mass="${mass}" x="0.3" y="0.08" z="0.03">
+                <origin xyz="0.0 0.0 0.0"/>
+            </xacro:inertial_box>
         </link>
+        <gazebo reference="${name}">
+            <material>
+                Gazebo/Orange
+            </material>
+        </gazebo>
     </xacro:macro>
     <!-- Rotor -->
-    <xacro:macro name="rotor" params="num parent radius length wing_pos">
+    <xacro:macro name="rotor" params="num parent radius length wing_pos mass">
         <joint name="rotor${num}_joint" type="continuous">
             <parent link="${parent}"/>
@@ -46,5 +56,13 @@
                 </geometry>
             </collision>
+            <xacro:inertial_cylinder mass="${mass}" length="${length}" radius="${radius}">
+                <origin xyz="0.0 0.0 0.0"/>
+            </xacro:inertial_cylinder>
         </link>
+        <gazebo reference="rotor${num}">
+            <material>
+                Gazebo/Blue
+            </material>
+        </gazebo>
     </xacro:macro>
 </robot>

File: src/my_robot_pkg/description/drone_macros.xacro (robot description, xacro)
@@ -4,5 +4,5 @@
     <xacro:property name = "mass" value = "1.0"/>
     <!-- Bar -->
-    <xacro:macro name="bar" params="name parent angle pos size ">
+    <xacro:macro name="bar" params="name parent angle pos size mass">
         <joint name="${name}_joint" type="fixed">
             <parent link="${parent}"/>
@@ -24,6 +24,8 @@
                 </geometry>
             </collision>
+            <xacro:inertial_box mass="${mass}" x="0.3" y="0.08" z="0.03">
+                <origin xyz="0.0 0.0 0.0"/>
+            </xacro:inertial_box>
         </link>
-        <xacro:inertial_box mass="${mass}" x="${size[0]}" y="${size[1]}" z="${size[2]}"></xacro:inertial_box>
         <gazebo reference="${name}">
             <material>
@@ -33,5 +35,5 @@
     </xacro:macro>
     <!-- Rotor -->
-    <xacro:macro name="rotor" params="num parent radius length wing_pos">
+    <xacro:macro name="rotor" params="num parent radius length wing_pos mass">
         <joint name="rotor${num}_joint" type="continuous">
             <parent link="${parent}"/>
@@ -54,8 +56,9 @@
                 </geometry>
             </collision>
+            <xacro:inertial_cylinder mass="${mass}" length="${length}" radius="${radius}">
+                <origin xyz="0.0 0.0 0.0"/>
+            </xacro:inertial_cylinder>
         </link>
-        <xacro:inertial_cylinder mass="${mass}" length="${length}" radius="${radius}">
-        </xacro:inertial_cylinder>
-        <gazebo>
+        <gazebo reference="rotor${num}">
             <material>
                 Gazebo/Blue
