Commit message: drone_diff_drive

File: install/my_robot_pkg/share/my_robot_pkg/description/gazebo_control.xacro (robot description, xacro)
@@ -9,5 +9,5 @@
             <wheel_diameter>0.1</wheel_diameter>
             <!-- Limits -->
-            <max_wheel_torque>50</max_wheel_torque>
+            <max_wheel_torque>5</max_wheel_torque>
             <max_wheel_acceleration>5.0</max_wheel_acceleration>
             <!-- Output -->

File: install/my_robot_pkg/share/my_robot_pkg/description/robot_core.xacro (robot description, xacro)
@@ -2,4 +2,5 @@
 <robot xmlns:xacro="https://www.ros.org/wiki/xacro" name="robot">
     <xacro:include filename="inertial_macros.xacro"/>
+    <xacro:property name="mass" value="0.5"/>
     <material name = "white">
         <color rgba="1 1 1 1"/>
@@ -37,5 +38,5 @@
             </geometry>
         </collision>
-        <xacro:inertial_box mass="0.5" x="0.3" y="0.3" z="0.15">
+        <xacro:inertial_box mass="${mass}" x="0.3" y="0.3" z="0.15">
             <origin xyz="0.15 0 0.075" rpy="0 0 0"/>
         </xacro:inertial_box>
@@ -65,5 +66,5 @@
             </geometry>
         </collision>
-        <xacro:inertial_cylinder mass="0.1" length="0.04" radius="0.05">
+        <xacro:inertial_cylinder mass="${mass}" length="0.04" radius="0.05">
             <origin xyz="0 0 0" rpy="0 0 0"/>
         </xacro:inertial_cylinder>
@@ -93,5 +94,5 @@
             </geometry>
         </collision>
-        <xacro:inertial_cylinder mass="0.1" length="0.04" radius="0.05">
+        <xacro:inertial_cylinder mass="${mass}" length="0.04" radius="0.05">
             <origin xyz="0 0 0" rpy="0 0 0"/>
         </xacro:inertial_cylinder>
@@ -120,5 +121,5 @@
             </geometry>
         </collision>
-        <xacro:inertial_sphere mass="0.1" radius="0.05">
+        <xacro:inertial_sphere mass="${mass}" radius="0.05">
             <origin xyz="0.0 0.0 0.0" rpy="0.0 0.0 0.0"/>
         </xacro:inertial_sphere>
